File: _schematics/v1.1.brd (EAGLE design)
At the start: 37 x 38 mm, 23 parts, among them J1 AC IN, U1 ESP-07, U2 MCP3221

Commit message: Update schematics
Parts:
- added ADC: (no value), jumper:SJ
- added R10: 220K, resistor:R0603
- added R11: 100K, resistor:R0603
- LED2: value RST -> RESET
- S1: device my_parts:SMD_BUTTON -> my_parts:TACTILE_SWITCH_SMD_6.2MM_TALL
- moved LED2 3.48 mm to (6.99, 35.7), turned to 90 degrees
- moved R4 3.14 mm to (8.26, 39.1)
- moved S1 1.57 mm to (3.33, 35.7), turned to 270 degrees
- moved J1 0.95 mm to (32.4, 35.9)
- moved PSU 0.64 mm to (15.9, 24.4)
- moved R1 0.48 mm to (8.10, 30.2)
Connections:
- new net N$4: ADC.1, R10.1, R11.1
- new net N$6: ADC.2, U1.2
- net ANALOG: now also R10.2
- net GND: now also R11.2, S1.A1, S1.A2; no longer S1.P$1, S1.P$3
- net RST: now also S1.B1, S1.B2; no longer S1.P$2, S1.P$4
Routing:
- net ANALOG: track 12.3 -> 18.4 mm, vias 0 -> 1
- net N$1: track 6.84 -> 2.36 mm
- net N$4: track 0.00 -> 4.45 mm
- net RST: track 13.1 -> 9.91 mm
- net N$6: track 0.00 -> 2.91 mm
- net VCC: track 28.1 -> 30.8 mm
- net GND: track 35.3 -> 36.1 mm
Other:
- board size 37 x 38 mm -> 37 x 39 mm

Commit message: [Schematics] Version 1.1 - Fix ADC polarity - Add input protection on programming header - Add voltage divider for RX signal
Connections:
- net RX: now also J4.1, U1.21; no longer J4.2, U1.22
- net TX: now also J4.2, U1.22; no longer J4.1, U1.21
Routing:
- net TX: track 30.1 -> 33.3 mm
- net RX: track 33.3 -> 30.1 mm
Other:
- board text added: "REV1.1"
- board text removed: "REV1"
Changed lines of the file:
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@@
 <setting verticaltext="up"/>
 </settings>
-<grid distance="6.25" unitdist="mil" unit="mil" style="lines" multiple="1" display="yes" altdistance="5" altunitdist="mil" altunit="mil"/>
+<grid distance="12.5" unitdist="mil" unit="mil" style="lines" multiple="1" display="yes" altdistance="5" altunitdist="mil" altunit="mil"/>
 <layers>
 <layer number="1" name="Top" color="4" fill="1" visible="yes" active="yes"/>
@@
 <wire x1="34.925" y1="35.2425" x2="34.925" y2="36.5125" width="0.0254" layer="20" curve="180"/>
 <wire x1="26.9875" y1="36.5125" x2="26.9875" y2="35.2425" width="0.0254" layer="20" curve="180"/>
-<text x="32.7025" y="2.54" size="1.27" layer="121" font="vector" ratio="12">REV1</text>
+<text x="36.5125" y="2.54" size="1.27" layer="121" font="vector" ratio="12" align="bottom-right">REV1.1</text>
 <wire x1="29.21" y1="31.4325" x2="34.6075" y2="31.4325" width="0.0254" layer="20"/>
 <wire x1="34.6075" y1="31.4325" x2="34.6075" y2="30.1625" width="0.0254" layer="20" curve="-180"/>
@@
 <wire x1="0.79375" y1="13.0175" x2="1.74625" y2="13.0175" width="0.15875" layer="121"/>
 <text x="1.42875" y="5.55625" size="0.9144" layer="121" font="vector" ratio="13" align="center">VCC</text>
-<text x="6.6675" y="5.55625" size="0.9144" layer="121" font="vector" ratio="13" align="center">RX</text>
-<text x="9.2075" y="5.55625" size="0.9144" layer="121" font="vector" ratio="13" align="center">TX</text>
+<text x="9.2075" y="5.55625" size="0.9144" layer="121" font="vector" ratio="13" align="center">RX</text>
+<text x="6.6675" y="5.55625" size="0.9144" layer="121" font="vector" ratio="13" align="center">TX</text>
 <text x="4.1275" y="5.55625" size="0.9144" layer="121" font="vector" ratio="13" align="center">GND</text>
 <text x="22.225" y="5.55625" size="0.9144" layer="121" font="vector" ratio="13" align="center">VCC</text>
@@
 <wire x1="30.265" y1="20.105" x2="30.48" y2="20.32" width="0.6096" layer="1"/>
 </signal>
-<signal name="RX">
+<signal name="TX">
 <contactref element="U1" pad="22"/>
 <contactref element="J4" pad="2"/>
@@
 <wire x1="22.55" y1="27.63" x2="24.298296875" y2="27.63" width="0.6096" layer="1"/>
 </signal>
-<signal name="TX">
+<signal name="RX">
 <contactref element="U1" pad="21"/>
 <contactref element="J4" pad="1"/>
