File: _schematics/v1.1.sch (EAGLE design)
At the start: 23 parts, among them J1 AC IN, U1 ESP-07, U2 MCP3221

Commit message: Update schematics
Parts:
- added ADC: (no value), jumper:SJ
- added R10: 220K, resistor:R-US_R0603
- added R11: 100K, resistor:R-US_R0603
- LED2: value RST -> RESET
- S1: device my_parts:BUTTONSMD -> my_parts:BUTTON
Connections:
- new net N$4: ADC.1, R10.1, R11.1
- new net N$6: ADC.2, U1.ADC
- net ANALOG: now also R10.2
- net GND: now also R11.2
Other:
- note added: "In case external ADC doesnt work"
Changed lines of the file:
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@@
 <part name="P+3" library="supply1" library_urn="urn:adsk.eagle:library:371" deviceset="VCC" device="" value="3V3"/>
 <part name="GND2" library="supply1" library_urn="urn:adsk.eagle:library:371" deviceset="GND" device=""/>
-<part name="S1" library="my_parts" library_urn="urn:adsk.eagle:library:225875" deviceset="BUTTON" device="SMD" package3d_urn="urn:adsk.eagle:package:2954938/2" value="RESET"/>
+<part name="S1" library="my_parts" library_urn="urn:adsk.eagle:library:225875" deviceset="BUTTON" device="" package3d_urn="urn:adsk.eagle:package:3123504/1" value="RESET"/>
 <part name="GND3" library="supply1" library_urn="urn:adsk.eagle:library:371" deviceset="GND" device=""/>
 <part name="R1" library="resistor" library_urn="urn:adsk.eagle:library:348" deviceset="R-US_" device="R0603" package3d_urn="urn:adsk.eagle:package:26057/1" value="10k"/>
@@
 <part name="GND5" library="supply1" library_urn="urn:adsk.eagle:library:371" deviceset="GND" device=""/>
 <part name="P+5" library="supply1" library_urn="urn:adsk.eagle:library:371" deviceset="VCC" device="" value="3V3"/>
-<part name="LED2" library="led" library_urn="urn:adsk.eagle:library:259" deviceset="LED" device="SML0805" package3d_urn="urn:adsk.eagle:package:15830/1" value="RST"/>
+<part name="LED2" library="led" library_urn="urn:adsk.eagle:library:259" deviceset="LED" device="SML0805" package3d_urn="urn:adsk.eagle:package:15830/1" value="RESET"/>
 <part name="R4" library="resistor" library_urn="urn:adsk.eagle:library:348" deviceset="R-US_" device="R0805" package3d_urn="urn:adsk.eagle:package:26059/1" value="100"/>
 <part name="J4" library="SparkFun-Connectors" library_urn="urn:adsk.eagle:library:513" deviceset="CONN_04" device="" package3d_urn="urn:adsk.eagle:package:38085/1"/>
@@
 <part name="R9" library="resistor" library_urn="urn:adsk.eagle:library:348" deviceset="R-US_" device="R0603" package3d_urn="urn:adsk.eagle:package:26057/1" value="2k"/>
 <part name="L1" library="resistor" library_urn="urn:adsk.eagle:library:348" deviceset="L-US" device="L2012C" package3d_urn="urn:adsk.eagle:package:25925/1" value="47nH"/>
+<part name="ADC" library="jumper" library_urn="urn:adsk.eagle:library:252" deviceset="SJ" device="" package3d_urn="urn:adsk.eagle:package:15471/1"/>
+<part name="R10" library="resistor" library_urn="urn:adsk.eagle:library:348" deviceset="R-US_" device="R0603" package3d_urn="urn:adsk.eagle:package:26057/1" value="220K"/>
+<part name="R11" library="resistor" library_urn="urn:adsk.eagle:library:348" deviceset="R-US_" device="R0603" package3d_urn="urn:adsk.eagle:package:26057/1" value="100K"/>
+<part name="GND1" library="supply1" library_urn="urn:adsk.eagle:library:371" deviceset="GND" device=""/>
 </parts>
 <sheets>
@@
 <plain>
 <text x="-25.4" y="2.54" size="1.778" layer="97">Either one of R2 or R3</text>
+<text x="5.08" y="-10.16" size="1.778" layer="97">In case external ADC doesnt work</text>
+<wire x1="15.24" y1="-7.62" x2="15.24" y2="12.7" width="0.1524" layer="97"/>
 </plain>
 <instances>
@@
 <instance part="R9" gate="G$1" x="10.16" y="35.56" rot="R180"/>
 <instance part="L1" gate="G$1" x="-15.24" y="60.96" rot="R180"/>
+<instance part="ADC" gate="1" x="15.24" y="15.24"/>
+<instance part="R10" gate="G$1" x="0" y="15.24" rot="R180"/>
+<instance part="R11" gate="G$1" x="7.62" y="7.62" rot="R270"/>
+<instance part="GND1" gate="1" x="7.62" y="-2.54"/>
 </instances>
 <busses>
@@
 <junction x="-12.7" y="27.94"/>
 </segment>
+<segment>
+<pinref part="R11" gate="G$1" pin="2"/>
+<wire x1="7.62" y1="2.54" x2="7.62" y2="0" width="0.1524" layer="91"/>
+<pinref part="GND1" gate="1" pin="GND"/>
+</segment>
 </net>
 <net name="RST" class="0">
@@
 <segment>
 <wire x1="-33.02" y1="22.86" x2="-22.86" y2="22.86" width="0.1524" layer="91"/>
-<wire x1="-22.86" y1="22.86" x2="-10.16" y2="22.86" width="0.1524" layer="91"/>
+<wire x1="-22.86" y1="22.86" x2="-15.24" y2="22.86" width="0.1524" layer="91"/>
 <pinref part="R2" gate="G$1" pin="2"/>
+<wire x1="-15.24" y1="22.86" x2="-10.16" y2="22.86" width="0.1524" layer="91"/>
 <wire x1="-22.86" y1="20.32" x2="-22.86" y2="22.86" width="0.1524" layer="91"/>
 <junction x="-22.86" y="22.86"/>
@@
 <pinref part="U2" gate="G$1" pin="A_IN"/>
 <label x="-33.02" y="22.86" size="1.778" layer="95"/>
+<wire x1="-15.24" y1="22.86" x2="-15.24" y2="15.24" width="0.1524" layer="91"/>
+<junction x="-15.24" y="22.86"/>
+<pinref part="R10" gate="G$1" pin="2"/>
+<wire x1="-15.24" y1="15.24" x2="-5.08" y2="15.24" width="0.1524" layer="91"/>
 </segment>
 </net>
@@
 </segment>
 </net>
+<net name="N$6" class="0">
+<segment>
+<pinref part="U1" gate="G$1" pin="ADC"/>
+<wire x1="30.48" y1="40.64" x2="27.94" y2="40.64" width="0.1524" layer="91"/>
+<wire x1="27.94" y1="40.64" x2="27.94" y2="15.24" width="0.1524" layer="91"/>
+<pinref part="ADC" gate="1" pin="2"/>
+<wire x1="20.32" y1="15.24" x2="27.94" y2="15.24" width="0.1524" layer="91"/>
+</segment>
+</net>
+<net name="N$4" class="0">
+<segment>
+<pinref part="R11" gate="G$1" pin="1"/>
+<pinref part="R10" gate="G$1" pin="1"/>
+<wire x1="5.08" y1="15.24" x2="7.62" y2="15.24" width="0.1524" layer="91"/>
+<wire x1="7.62" y1="15.24" x2="7.62" y2="12.7" width="0.1524" layer="91"/>
+<pinref part="ADC" gate="1" pin="1"/>
+<wire x1="7.62" y1="15.24" x2="10.16" y2="15.24" width="0.1524" layer="91"/>
+<junction x="7.62" y="15.24"/>
+</segment>
+</net>

Commit message: [Schematics] Version 1.1 - Fix ADC polarity - Add input protection on programming header - Add voltage divider for RX signal
Connections:
- net RX: now also J4.1, U1.RXD0/IO3; no longer J4.2, U1.TXD0/IO1
- net TX: now also J4.2, U1.TXD0/IO1; no longer J4.1, U1.RXD0/IO3
Changed lines of the file:
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@@
 </segment>
 </net>
-<net name="RX" class="0">
+<net name="TX" class="0">
 <segment>
 <wire x1="68.58" y1="43.18" x2="68.58" y2="55.88" width="0.1524" layer="91"/>
@@
 </segment>
 </net>
-<net name="TX" class="0">
+<net name="RX" class="0">
 <segment>
 <wire x1="66.04" y1="58.42" x2="96.52" y2="58.42" width="0.1524" layer="91"/>
